File: BF@kicad/bf-025.kicad_pcb (KiCad board)
At the start: 2 copper layers, 100 x 100 mm, 578 parts, among them J101 Barrel_Jack_Switch, J102 I2C, J103 UART, U101 M5Atom

Commit message: PCB data
footprint, 3d-omage
Parts:
- REF** (x8): footprint BF:BF@MouseBite_r48_50 -> bf:BF@MouseBite_r48_50

Commit message: V03L02
update PCB
Parts:
- moved D101 2.50 mm to (2.50, -20.8)
Routing:
- net GND: track 1879.3 -> 1898.9 mm, vias 367 -> 359
- net +5V: track 2138.9 -> 2141.2 mm
- net /M5_5V: track 24.7 -> 25.9 mm
- net /WS2812C_60_2/DIN: track 7.47 -> 8.20 mm
Other:
- board text added: "BF-025 V03L02 RGB-LED Clock 276 for M5Atom Copyright 2021"
- board text removed: "BF-025 V03L01 RGB-LED Clock 276 for M5Atom Copyright 2021"
